Commit message: Add a steering angle in the buggy urdf description.

File: data/urdf/buggy.urdf (robot description, URDF)
Before this commit: robot buggy, 1 links, 0 joints
Joints:
- added joint steering angle: type revolute, parent base_link, origin xyz=1.36 0 0 rpy=0 0 0, axis 0 0 1, limit lower=-1 upper=1

Commit message: Add a link for steering wheel in urdf file.

File: data/urdf/buggy.urdf (robot description, URDF)
Before this commit: robot buggy, 1 links, 1 joints
Links:
- added link virtual_front_wheel; visual cylinder length=.1 radius=.1
Joints:
- joint steering angle: child (none) -> virtual_front_wheel; limit lower=-1 upper=1 -> lower=-1 upper=1 effort=10 velocity=1

Commit message: Finish implementation of steering method
  - fix some compilation and execution bugs,
  - add debug output.

File: data/urdf/buggy.urdf (robot description, URDF)
Before this commit: robot buggy, 2 links, 1 joints
Links:
- link virtual_front_wheel: geometry visual cylinder length=.01 radius=.01
